File: Hardware/Design/SolarPwrOption_open.sch (EAGLE design)
At the start: 8 parts, among them Q2 DMP4065S, Q3 BSS138, U2 OKI-78SR-5/1.5-W36-C

Commit message: Hardware: 30w pv is to much for alt input
Other:
- note added: "1.31A (Isc)"
- note added: "13AHr"
- note added: "SLP020-12U"
- note removed: "1.74A (Isc)"
- note removed: "17AHr"
- note removed: "SLP030-12U"
Changed lines of the file:
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@@
 <wire x1="5.08" y1="7.62" x2="5.08" y2="43.18" width="0.1524" layer="98"/>
 <text x="8.128" y="40.64" size="1.778" layer="98">ON CIRCUIT BOARD</text>
-<text x="79.248" y="41.656" size="1.778" layer="98">SLP030-12U</text>
-<text x="86.868" y="27.94" size="1.778" layer="98">1.74A (Isc)</text>
+<text x="79.248" y="41.656" size="1.778" layer="98">SLP020-12U</text>
+<text x="86.868" y="27.94" size="1.778" layer="98">1.31A (Isc)</text>
 <text x="86.868" y="33.02" size="1.778" layer="98">21.6V (Voc)</text>
 <text x="74.168" y="16.002" size="1.778" layer="98">LA</text>
 <text x="74.168" y="12.7" size="1.778" layer="98">12V</text>
-<text x="74.168" y="9.398" size="1.778" layer="98">17AHr</text>
+<text x="74.168" y="9.398" size="1.778" layer="98">13AHr</text>
 <text x="7.112" y="23.622" size="1.778" layer="98">AVR PIN</text>
 <text x="79.248" y="38.608" size="1.778" layer="98">WITHOUT BY-PASS DIODES</text>
